File: forRaspberryPi3/rpi3GpioTester/rpi3GpioTester.kicad_pcb (KiCad board)
At the start: 2 copper layers, 78.7 x 119.4 mm, 63 parts, among them J1 Raspberry_Pi_2_3, J2 Conn_01x20_Male, J3 Conn_01x12_Male, SW12 SW_Push, SW13 SW_Push, SW16 SW_Push, SW17 SW_Push, SW18 SW_Push, SW19 SW_Push, SW20 SW_Push, SW21 SW_Push, SW22 SW_Push, SW23 SW_Push, SW24 SW_Push, SW25 SW_Push, SW26 SW_Push, SW27 SW_Push, SW4 SW_Push, SW5 SW_Push, SW6 SW_Push

Commit message: Update rpi3GpioTester pcb design
Other:
- outline, holes or cut-outs redrawn
Changed lines of the file:
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@@
   (general
     (thickness 1.6)
-    (drawings 41)
+    (drawings 57)
     (tracks 591)
     (zones 0)
@@
     )
   )
+  (gr_line (start 76.835 95.885) (end 76.835 146.685) (layer F.SilkS) (width 0.15))
+  (gr_line (start 78.105 94.615) (end 76.835 95.885) (layer F.SilkS) (width 0.15))
+  (gr_line (start 83.185 94.615) (end 78.105 94.615) (layer F.SilkS) (width 0.15))
+  (gr_line (start 83.185 146.685) (end 83.185 94.615) (layer F.SilkS) (width 0.15))
+  (gr_line (start 76.835 146.685) (end 83.185 146.685) (layer F.SilkS) (width 0.15))
+  (gr_line (start 86.995 86.995) (end 112.395 86.995) (layer F.SilkS) (width 0.15))
+  (gr_line (start 86.995 71.755) (end 86.995 86.995) (layer F.SilkS) (width 0.15))
+  (gr_line (start 93.345 71.755) (end 86.995 71.755) (layer F.SilkS) (width 0.15))
+  (gr_line (start 102.235 71.755) (end 112.395 71.755) (layer F.SilkS) (width 0.15))
+  (gr_line (start 86.995 107.315) (end 112.395 107.315) (layer F.SilkS) (width 0.15))
+  (gr_line (start 86.995 92.075) (end 86.995 107.315) (layer F.SilkS) (width 0.15))
+  (gr_line (start 93.345 92.075) (end 86.995 92.075) (layer F.SilkS) (width 0.15))
+  (gr_line (start 102.235 92.075) (end 112.395 92.075) (layer F.SilkS) (width 0.15))
+  (gr_arc (start 36.83 31.75) (end 36.83 29.21) (angle -90) (layer Edge.Cuts) (width 0.15))
+  (gr_arc (start 36.83 146.05) (end 34.29 146.05) (angle -90) (layer Edge.Cuts) (width 0.15))
+  (gr_arc (start 110.49 146.05) (end 110.49 148.59) (angle -90) (layer Edge.Cuts) (width 0.15))
+  (gr_arc (start 110.49 31.75) (end 113.03 31.75) (angle -90) (layer Edge.Cuts) (width 0.15))
   (gr_text "CHIRIMEN Open Hardware\nCommunity" (at 43.18 133.35 90) (layer F.SilkS)
     (effects (font (size 1.5 1.5) (thickness 0.3)))
@@
     (effects (font (size 1.5 1.5) (thickness 0.3)))
   )
-  (gr_text "I2C : B" (at 97.79 92.075) (layer F.SilkS)
+  (gr_text "I2C : A" (at 97.79 92.075) (layer F.SilkS)
     (effects (font (size 1.5 1.5) (thickness 0.3)))
   )
@@
     (effects (font (size 1.5 1.5) (thickness 0.3)))
   )
-  (gr_text "I2C : A" (at 97.79 71.755) (layer F.SilkS)
+  (gr_text "I2C : B" (at 97.79 71.755) (layer F.SilkS)
     (effects (font (size 1.5 1.5) (thickness 0.3)))
   )
@@
     (effects (font (size 1.5 1.5) (thickness 0.3)))
   )
-  (gr_line (start 34.29 29.21) (end 34.29 29.845) (angle 90) (layer Edge.Cuts) (width 0.15))
-  (gr_line (start 113.03 29.21) (end 34.29 29.21) (angle 90) (layer Edge.Cuts) (width 0.15))
-  (gr_line (start 113.03 148.59) (end 113.03 29.21) (angle 90) (layer Edge.Cuts) (width 0.15))
-  (gr_line (start 34.29 148.59) (end 113.03 148.59) (angle 90) (layer Edge.Cuts) (width 0.15))
-  (gr_line (start 34.29 29.845) (end 34.29 148.59) (angle 90) (layer Edge.Cuts) (width 0.15))
+  (gr_line (start 110.49 29.21) (end 36.83 29.21) (angle 90) (layer Edge.Cuts) (width 0.15))
+  (gr_line (start 113.03 146.05) (end 113.03 31.75) (angle 90) (layer Edge.Cuts) (width 0.15))
+  (gr_line (start 36.83 148.59) (end 110.49 148.59) (angle 90) (layer Edge.Cuts) (width 0.15))
+  (gr_line (start 34.29 31.75) (end 34.29 146.05) (angle 90) (layer Edge.Cuts) (width 0.15))
   (segment (start 93.98 55.88) (end 97.79 55.88) (width 0.25) (layer F.Cu) (net 1))
   (segment (start 86.36 55.88) (end 93.98 55.88) (width 0.25) (layer F.Cu) (net 1))

Commit message: rpi3GpioTester rev0.3
Parts:
- added I2C10: Conn_01x04_Female, Socket_Strips:Socket_Strip_Straight_1x04_Pitch2.54mm, F.Cu at (99.1, 81.3)
- added I2C11: Conn_01x04_Female, Socket_Strips:Socket_Strip_Straight_1x04_Pitch2.54mm, F.Cu at (99.1, 75.6)
- added I2C12: Conn_01x04_Female, Socket_Strips:Socket_Strip_Straight_1x04_Pitch2.54mm, F.Cu at (99.1, 69.8)
- added I2C13: Conn_01x04_Female, Socket_Strips:Socket_Strip_Straight_1x04_Pitch2.54mm, F.Cu at (99.1, 64.1)
- added I2C14: Conn_01x04_Female, Socket_Strips:Socket_Strip_Straight_1x04_Pitch2.54mm, F.Cu at (99.1, 58.4)
- added I2C15: Conn_01x04_Female, Socket_Strips:Socket_Strip_Straight_1x04_Pitch2.54mm, F.Cu at (99.1, 52.7)
- added I2C16: Conn_01x04_Female, Socket_Strips:Socket_Strip_Straight_1x04_Pitch2.54mm, F.Cu at (99.1, 47.0)
- added I2C9: Conn_01x04_Female, Socket_Strips:Socket_Strip_Straight_1x04_Pitch2.54mm, F.Cu at (99.1, 87.0)
- added I2C_Grove2: Conn_01x04, Connectors:Grove_1x04, F.Cu at (88.3, 69.2)
- added I2C_Grove3: Conn_01x04, Connectors:Grove_1x04, F.Cu at (88.3, 77.5)
- added I2C_Grove4: Conn_01x04, Connectors:Grove_1x04, F.Cu at (88.3, 85.7)
- moved I2C1 43.6 mm to (99.1, 139.1), turned to 90 degrees
- moved I2C5 41.1 mm to (99.1, 116.2), turned to 90 degrees
- moved I2C2 37.0 mm to (99.1, 133.3), turned to 90 degrees
- moved I2C6 34.5 mm to (99.1, 110.5), turned to 90 degrees
- moved I2C3 31.2 mm to (99.1, 127.6), turned to 90 degrees
- moved I2C7 28.6 mm to (99.1, 104.8), turned to 90 degrees
- moved I2C4 26.5 mm to (99.1, 121.9), turned to 90 degrees
- moved I2C8 24.1 mm to (99.1, 99.1), turned to 90 degrees
- moved I2C_Grove1 16.8 mm to (88.3, 61.0), turned to 270 degrees
- moved D6 13.6 mm to (91.4, 54.0)
- moved R6 13.6 mm to (76.8, 51.4)
- moved SW6 13.6 mm to (80.0, 48.9)
- moved D5 12.0 mm to (91.4, 45.7)
- moved R5 12.0 mm to (76.8, 43.2)
- moved SW5 12.0 mm to (80.0, 40.6)
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Connections:
- I2C5 pad 1: GND -> SDA
- I2C5 pad 3: SDA -> GND
- I2C6 pad 1: GND -> SDA
- I2C6 pad 3: SDA -> GND
- I2C7 pad 1: GND -> SDA
- I2C7 pad 3: SDA -> GND
- I2C8 pad 1: GND -> SDA
- I2C8 pad 3: SDA -> GND
Routing:
- net SDA: track 73.7 -> 216.4 mm
- net SCL: track 78.9 -> 213.6 mm
- net +3V3: track 521.1 -> 589.9 mm, vias 5 -> 8
- net G5: track 156.6 -> 162.9 mm
- net GND: track 57.2 -> 61.5 mm, vias 0 -> 1
- net G4: track 138.3 -> 142.6 mm
- net SPI_CE1: track 17.6 -> 13.4 mm, vias 0 -> 1
- net SPI_CE0: track 19.7 -> 15.5 mm, vias 1 -> 2
- net RXD0: track 30.1 -> 26.4 mm
- net TXD0: track 30.9 -> 27.9 mm
- net SPI_MISO: track 24.7 -> 22.8 mm
- net +5V: track 98.4 -> 97.2 mm, vias 6 -> 5
- net SPI_SCLK: track 25.4 -> 26.1 mm
- net ID_SD: track 25.4 -> 26.1 mm
- net SPI_MOSI: track 28.3 -> 28.6 mm, vias 0 -> 3
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Other:
- board text added: "GND 3V3 SDA SCL"
- board text removed: "SCL SDA 3V3 GND"

Commit message: Add I2C pull up pattern
Parts:
- added I2C_PU1: Conn_01x04_Female, Socket_Strips:Socket_Strip_Straight_1x04_Pitch2.54mm, F.Cu at (99.1, 38.1)
- added J_5V1: Conn_01x04_Female, Socket_Strips:Socket_Strip_Straight_1x04_Pitch2.54mm, F.Cu at (88.9, 102.9)
- added J_GND1: Conn_01x04_Female, Socket_Strips:Socket_Strip_Straight_1x04_Pitch2.54mm, F.Cu at (92.7, 102.9)
- moved I2C10 1.91 mm to (99.1, 83.2)
- moved I2C11 1.91 mm to (99.1, 77.5)
- moved I2C12 1.91 mm to (99.1, 71.8)
- moved I2C13 1.91 mm to (99.1, 66.0)
- moved I2C14 1.91 mm to (99.1, 60.3)
- moved I2C15 1.91 mm to (99.1, 54.6)
- moved I2C16 1.91 mm to (99.1, 48.9)
- moved I2C9 1.91 mm to (99.1, 88.9)
Routing:
- net +3V3: track 589.9 -> 604.1 mm
- net +5V: track 97.2 -> 107.4 mm
- net SDA: track 216.4 -> 224.9 mm
- net SCL: track 213.6 -> 220.7 mm
Other:
- board text added: "3V3"
- board text added: "SCL"
- board text added: "SDA"

Commit message: Minor update
Parts:
- moved I2C_Grove1 24.8 mm to (88.3, 85.7)
- moved I2C_Grove4 24.8 mm to (88.3, 61.0)
- moved I2C_Grove2 8.25 mm to (88.3, 77.5)
- moved I2C_Grove3 8.25 mm to (88.3, 69.2)
Changed lines of the file:
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@@
   )
   (module Connectors:Grove_1x04 (layer F.Cu)
-    (at 88.265 85.725 270)
+    (at 88.265 60.96 270)
     (descr https://statics3.seeedstudio.com/images/opl/datasheet/3470130P1.pdf)
     (tags Grove-1x04)
-    (fp_text reference I2C_Grove4 (at 1.27 -3.81 90) (layer F.SilkS)
+    (fp_text reference I2C_Grove4 (at -0.635 -3.81 90) (layer F.SilkS)
       (effects (font (size 1 1) (thickness 0.15)))
     )
@@
   )
   (module Connectors:Grove_1x04 (layer F.Cu)
-    (at 88.265 69.215 270)
+    (at 88.265 77.47 270)
     (descr https://statics3.seeedstudio.com/images/opl/datasheet/3470130P1.pdf)
     (tags Grove-1x04)
-    (fp_text reference I2C_Grove2 (at 0 -3.81 90) (layer F.SilkS)
+    (fp_text reference I2C_Grove2 (at 0.635 -3.81 90) (layer F.SilkS)
       (effects (font (size 1 1) (thickness 0.15)))
     )
@@
   )
   (module Connectors:Grove_1x04 (layer F.Cu)
-    (at 88.265 77.47 270)
+    (at 88.265 69.215 270)
     (descr https://statics3.seeedstudio.com/images/opl/datasheet/3470130P1.pdf)
     (tags Grove-1x04)
-    (fp_text reference I2C_Grove3 (at 0.635 -3.81 90) (layer F.SilkS)
+    (fp_text reference I2C_Grove3 (at 0 -3.81 90) (layer F.SilkS)
       (effects (font (size 1 1) (thickness 0.15)))
     )
@@
   )
   (module Connectors:Grove_1x04 (layer F.Cu)
-    (at 88.265 60.96 270)
+    (at 88.265 85.725 270)
     (descr https://statics3.seeedstudio.com/images/opl/datasheet/3470130P1.pdf)
     (tags Grove-1x04)
-    (fp_text reference I2C_Grove1 (at -0.635 -3.81 90) (layer F.SilkS)
-      (effects (font (size 1 1) (thickness 0.15)))
-    )
+    (fp_text reference I2C_Grove1 (at 1.27 -3.81 90) (layer F.SilkS)
+      (effects (font (size 1 1) (thickness 0.15)))
+    )
